File: Kicad/MidiMapper.sch (KiCad schematic (older format))
At the start: 35 parts, among them IC1 74LS07N, IC2 74LS07N, P1 IN, P2 THRU, P3 OUT1, P4 OUT2, P5 OUT3, P6 OUT4

Commit message: New RealtimePage layout and some screen navigation fixes.
Parts:
- removed C1, C2: 100nF, ~, symbol C
- removed D1: 1N4148, ~, symbol DIODE
- removed R1, R10, R11, R12, R13, R14, R15, R16, R17, R18, R4, R5, R6, R7, R8, R9: 220, ~, symbol R
- removed R2: 100k, ~, symbol R
- removed R3: 10k, ~, symbol R
- added C? (x2): 18p, symbol C_Small
- added C? (x2): C_Small, symbol C_Small
- added CON?: AVR-JTAG-10, AVR-JTAG-10, symbol AVR-JTAG-10
- added D1, D? (x8): 1N4148, symbol D
- added IC?: ATMEGA1284-P, DIL40, symbol ATMEGA1284-P
- added P?: CONN_02X08, symbol CONN_02X08
- added R? (x16): 220, symbol R
- added R? (x2): 10k, symbol R
- added R?: 100k, symbol R
- added R? (x4): 5k6, symbol R
- added RV?: POT, symbol POT
- added SW?: Left, symbol SW_PUSH_SMALL
- added SW?: Right, symbol SW_PUSH_SMALL
- added SW?: Up, symbol SW_PUSH_SMALL
- added SW?: Down, symbol SW_PUSH_SMALL
- added SW?: Enter, symbol SW_PUSH_SMALL
- added SW?: Exit, symbol SW_PUSH_SMALL
- added SW?: s1, symbol SW_PUSH_SMALL
- added SW?: s2, symbol SW_PUSH_SMALL
- added Y?: 20MHz, symbol Crystal
- D2, D3, D4, D5, D6: symbol LED -> LED-RESCUE-MidiMapper
Connections:
- net labels added: D0/4, D1/5, D2/6, D3/7, E, KeyRow0, KeyRow1, KeyScan0, KeyScan1, KeyScan2, KeyScan3, LCD-Contrast, MIDI-IN, MIDI-OUT1, MIDI-OUT2, MIDI-OUT3, MIDI-OUT4, RESET, RS, TCK, TDI, TDO, TMS
- wire segments 69 -> 253
Other:
- note added: "AVR-JTAG"
- note added: "Key Pad"
- note added: "LCD"
- moved on the sheet: IC1G, IC2A, IC2G, OC1

Commit message: rescued
Parts:
- added C? (x3): 100n, symbol C_Small
- added C?: 47u, symbol CP_Small
- added P?: CONN_01X16, symbol CONN_01X16
- C? (x2): value C_Small -> 100n
- RV?: value POT -> 10k
Connections:
- wire segments 253 -> 289
